File: 50x50_protoboard.sch (KiCad schematic (older format))
At the start: 89 parts, among them CON1 BARREL_JACK, CON2 USB-MINI-B, CON3 USB-MICRO, J1 INTERCONNECT_3X1, J10 INTERCONNECT_3X1, J11 INTERCONNECT_3X1, J12 INTERCONNECT_3X1, J13 INTERCONNECT_3X1, J14 INTERCONNECT_3X1, J15 INTERCONNECT_3X1, J16 INTERCONNECT_3X1, J17 INTERCONNECT_3X1, J18 INTERCONNECT_3X1, J19 INTERCONNECT_3X1, J2 INTERCONNECT_3X1, J20 INTERCONNECT_3X1, J21 INTERCONNECT_3X1, J22 INTERCONNECT_3X1, J23 INTERCONNECT_3X1, J24 INTERCONNECT_3X1, J25 INTERCONNECT_3X1, J26 INTERCONNECT_3X1, J27 INTERCONNECT_3X1, J28 INTERCONNECT_3X1, J29 INTERCONNECT_3X1, J3 INTERCONNECT_3X1, J30 INTERCONNECT_3X1, J31 INTERCONNECT_3X1, J32 INTERCONNECT_3X1, J33 INTERCONNECT_3X1, J34 INTERCONNECT_3X1, J35 INTERCONNECT_3X1, J36 INTERCONNECT_3X1, J37 INTERCONNECT_3X1, J38 INTERCONNECT_3X1, J39 INTERCONNECT_3X1, J4 INTERCONNECT_3X1, J40 INTERCONNECT_3X1, J41 INTERCONNECT_3X1, J42 INTERCONNECT_3X1, J43 INTERCONNECT_3X1, J44 INTERCONNECT_3X1, J45 INTERCONNECT_3X1, J46 INTERCONNECT_3X1, J47 INTERCONNECT_3X1, J48 INTERCONNECT_3X1, J49 INTERCONNECT_3X1, J5 INTERCONNECT_3X1, J50 INTERCONNECT_3X1, J51 INTERCONNECT_3X1, J52 INTERCONNECT_3X1, J53 INTERCONNECT_3X1, J54 INTERCONNECT_3X1, J55 INTERCONNECT_3X1, J56 INTERCONNECT_3X1, J57 INTERCONNECT_3X1, J58 INTERCONNECT_3X1, J59 INTERCONNECT_3X1, J6 INTERCONNECT_3X1, J60 INTERCONNECT_3X1, J61 INTERCONNECT_3X1, J62 INTERCONNECT_3X1, J63 INTERCONNECT_3X1, J64 INTERCONNECT_3X1, J65 INTERCONNECT_2X1, J7 INTERCONNECT_3X1, J8 INTERCONNECT_3X1, J9 INTERCONNECT_3X1, P1 CONN_5, U1 7805

Commit message: switched to UNLICENSE and updated modules and directory structure to that of newer kicad projects
Parts:
- removed CON2: USB-MINI-B, ~, symbol USB-MINI-B
- removed CON3: USB-MICRO, ~, symbol USB-MINI-B
- removed U1: 7805, ~, symbol 7805
- removed VIN1, VIN_78XX1: INTERCONNECT_4X1, ~, symbol INTERCONNECT_4X1
- removed VIN2, VOUT_78XX1: INTERCONNECT_6X1, ~, symbol INTERCONNECT_6X1
- added CON2, CON3: USB_FEMALE_WITH_ID, symbol USB_FEMALE_WITH_ID
- added U1: LM7805CT, TO-220, symbol LM7805CT
- added VIN1, VIN_78XX1: CONN_4, symbol CONN_4
- added VIN2, VOUT_78XX1: CONN_6, symbol CONN_6
Connections:
- wire segments 118 -> 117
Other:
- moved on the sheet: C1, C2, CON1, F1, F2, GND1, GND2, GND3, J1, J10, J11, J12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

Commit message: added screw hole, moved fuse to VIN instead of GND and rounded the outline corners
Parts:
- added JP7: JUMPER, symbol JUMPER
- VIN1, VIN_78XX1: value CONN_4 -> CONN_2; symbol CONN_4 -> CONN_2
Connections:
- net at C1.2, C2.2, GND1.1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: now also JP7.2; no longer F1.2, F2.2, JP1.2
- net at JP2.1, JP3.1: now also F1.2, F2.2, JP1.2; no longer CON1.1
- net at F1.1, F2.1, JP1.1: now also CON1.1; no longer CON1.2
- net at C1.1, JP2.2, U1.1 (IN)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: no longer VIN_78XX1.3 (P3), VIN_78XX1.4 (P4)
- net at JP3.2, JP4.2, JP5.2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: no longer VIN1.3 (P3), VIN1.4 (P4)
- new net: CON1.2, JP7.1
Other:
- moved on the sheet: CON1, F1, F2, J65, JP1
Changed lines of the file:
@@
 L BARREL_JACK CON1
 U 1 1 53DD4216
-P 1450 1300
-F 0 "CON1" H 1450 1550 60  0000 C CNN
-F 1 "BARREL_JACK" H 1450 1100 60  0000 C CNN
-F 2 "~" H 1450 1300 60  0000 C CNN
-F 3 "~" H 1450 1300 60  0000 C CNN
-	1    1450 1300
+P 1550 2250
+F 0 "CON1" H 1550 2500 60  0000 C CNN
+F 1 "BARREL_JACK" H 1550 2050 60  0000 C CNN
+F 2 "~" H 1550 2250 60  0000 C CNN
+F 3 "~" H 1550 2250 60  0000 C CNN
+	1    1550 2250
 	1    0    0    -1
 $EndComp
@@
 L JUMPER JP1
 U 1 1 53DD424D
-P 1450 1850
-F 0 "JP1" H 1450 2000 60  0000 C CNN
-F 1 "JUMPER" H 1450 1770 40  0000 C CNN
-F 2 "~" H 1450 1850 60  0000 C CNN
-F 3 "~" H 1450 1850 60  0000 C CNN
-	1    1450 1850
+P 1700 1200
+F 0 "JP1" H 1700 1350 60  0000 C CNN
+F 1 "JUMPER" H 1700 1120 40  0000 C CNN
+F 2 "~" H 1700 1200 60  0000 C CNN
+F 3 "~" H 1700 1200 60  0000 C CNN
+	1    1700 1200
 	1    0    0    -1
 $EndComp
@@
 L INTERCONNECT_2X1 J65
 U 1 1 53DD425C
-P 2050 1500
-F 0 "J65" H 2050 1600 60  0000 C CNN
-F 1 "INTERCONNECT_2X1" H 2050 1400 60  0001 C CNN
-F 2 "~" H 2050 1500 60  0000 C CNN
-F 3 "~" H 2050 1500 60  0000 C CNN
-	1    2050 1500
+P 2150 2250
+F 0 "J65" H 2150 2350 60  0000 C CNN
+F 1 "INTERCONNECT_2X1" H 2150 2150 60  0001 C CNN
+F 2 "~" H 2150 2250 60  0000 C CNN
+F 3 "~" H 2150 2250 60  0000 C CNN
+	1    2150 2250
 	1    0    0    -1
 $EndComp
@@
 L FUSE F1
 U 1 1 53DDB6F8
-P 1400 2100
-F 0 "F1" H 1500 2150 40  0000 C CNN
-F 1 "FUSE" H 1300 2050 40  0000 C CNN
-F 2 "~" H 1400 2100 60  0000 C CNN
-F 3 "~" H 1400 2100 60  0000 C CNN
-	1    1400 2100
+P 1650 1450
+F 0 "F1" H 1750 1500 40  0000 C CNN
+F 1 "FUSE" H 1550 1400 40  0000 C CNN
+F 2 "~" H 1650 1450 60  0000 C CNN
+F 3 "~" H 1650 1450 60  0000 C CNN
+	1    1650 1450
 	1    0    0    -1
 $EndComp
@@
 L FUSE F2
 U 1 1 53DDB707
-P 1400 2350
-F 0 "F2" H 1500 2400 40  0000 C CNN
-F 1 "FUSE" H 1300 2300 40  0000 C CNN
-F 2 "~" H 1400 2350 60  0000 C CNN
-F 3 "~" H 1400 2350 60  0000 C CNN
-	1    1400 2350
+P 1650 1700
+F 0 "F2" H 1750 1750 40  0000 C CNN
+F 1 "FUSE" H 1550 1650 40  0000 C CNN
+F 2 "~" H 1650 1700 60  0000 C CNN
+F 3 "~" H 1650 1700 60  0000 C CNN
+	1    1650 1700
 	1    0    0    -1
 $EndComp
@@
 $EndComp
 $Comp
-L CONN_4 VIN_78XX1
+L CONN_2 VIN_78XX1
 U 1 1 554BC195
 P 3150 850
 F 0 "VIN_78XX1" V 3100 850 50  0000 C CNN
-F 1 "CONN_4" V 3200 850 50  0000 C CNN
+F 1 "CONN_2" V 3200 850 50  0000 C CNN
 F 2 "" H 3150 850 60  0000 C CNN
 F 3 "" H 3150 850 60  0000 C CNN
@@
 $EndComp
 $Comp
-L CONN_4 VIN1
+L CONN_2 VIN1
 U 1 1 554BCE60
-P 3200 1450
-F 0 "VIN1" V 3150 1450 50  0000 C CNN
-F 1 "CONN_4" V 3250 1450 50  0000 C CNN
-F 2 "" H 3200 1450 60  0000 C CNN
-F 3 "" H 3200 1450 60  0000 C CNN
-	1    3200 1450
+P 3150 1450
+F 0 "VIN1" V 3100 1450 50  0000 C CNN
+F 1 "CONN_2" V 3200 1450 50  0000 C CNN
+F 2 "" H 3150 1450 60  0000 C CNN
+F 3 "" H 3150 1450 60  0000 C CNN
+	1    3150 1450
 	0    -1   -1   0
 $EndComp
@@
 Connection ~ 3850 4300
 Connection ~ 3050 4350
-Connection ~ 3050 1800
-Connection ~ 3150 1800
-Connection ~ 3250 1800
-Connection ~ 3350 1800
 Connection ~ 4400 1800
 Connection ~ 4500 1800
@@
 Wire Wire Line
 	2850 1200 3450 1200
-Connection ~ 3000 1200
-Connection ~ 3100 1200
-Connection ~ 3200 1200
-Connection ~ 3300 1200
 Wire Wire Line
 	4250 1200 4900 1200
@@
 Connection ~ 4700 1200
 Connection ~ 4800 1200
-Wire Wire Line
-	1750 1400 1750 1600
-Wire Wire Line
-	1750 1600 1150 1600
-Wire Wire Line
-	1150 1600 1150 2350
 Connection ~ 3850 2800
 Wire Wire Line
@@
 Wire Wire Line
 	2700 2900 2450 2900
-Connection ~ 1150 1850
-Connection ~ 1150 2100
-Wire Wire Line
-	1650 2350 1650 2100
-Wire Wire Line
-	1650 2100 3050 2100
+Connection ~ 1400 1450
+Wire Wire Line
+	1900 1700 1900 1450
 Wire Wire Line
 	1800 4500 2700 4500
@@
 Connection ~ 4550 2800
 Connection ~ 3750 2800
-Connection ~ 1750 2100
 Connection ~ 3050 2800
 Wire Wire Line
 	4900 1800 2850 1800
 Wire Wire Line
-	3350 1950 3350 1800
-Wire Wire Line
 	4900 2100 4900 1800
 Wire Wire Line
@@
 Wire Wire Line
 	4250 1300 4250 1200
-Wire Wire Line
-	3050 2100 3050 4350
 Wire Wire Line
 	3450 1300 3550 1300
@@
 	4900 2100 4550 2100
 Wire Wire Line
-	3750 2100 3750 1950
-Wire Wire Line
-	3750 1950 3350 1950
+	3750 1950 3750 2100
+Wire Wire Line
+	3250 1950 3750 1950
 Connection ~ 2250 1200
-Wire Wire Line
-	1750 1200 2250 1200
-Wire Wire Line
-	2250 1200 2250 1800
-Wire Wire Line
-	1750 1300 1900 1300
-Wire Wire Line
-	1900 1300 1900 1500
-Wire Wire Line
-	1900 1500 2100 1500
-Connection ~ 2000 1500
-Wire Wire Line
-	1750 2100 1750 1850
+Connection ~ 2100 2250
 Wire Wire Line
 	2650 3000 2650 4350
@@
 Connection ~ 2450 3200
 Connection ~ 2450 3300
+Wire Wire Line
+	1850 2250 2200 2250
+Connection ~ 1900 1450
+Connection ~ 2000 1200
+Wire Wire Line
+	2000 1200 2000 1450
+Wire Wire Line
+	2000 1450 1900 1450
+Wire Wire Line
+	2000 1200 2250 1200
+Wire Wire Line
+	2250 1200 2250 1800
+Wire Wire Line
+	1400 1200 1400 1850
+Wire Wire Line
+	1400 1850 1850 1850
+Wire Wire Line
+	1850 1850 1850 2150
+Connection ~ 1400 1700
+$Comp
+L JUMPER JP7
+U 1 1 554BE7A5
+P 2750 2350
+F 0 "JP7" H 2750 2500 60  0000 C CNN
+F 1 "JUMPER" H 2750 2270 40  0000 C CNN
+F 2 "" H 2750 2350 60  0000 C CNN
+F 3 "" H 2750 2350 60  0000 C CNN
+	1    2750 2350
+	1    0    0    -1
+$EndComp
+Wire Wire Line
+	1850 2350 2450 2350
+Wire Wire Line
+	3050 2350 3050 4350
+Connection ~ 3250 1200
+Connection ~ 3050 1200
+Connection ~ 3050 1800
+Connection ~ 3250 1800
+Wire Wire Line
+	3250 1800 3250 1950
 $EndSCHEMATC

Commit message: created interconnect schematic symbols in 2.54mm_Pin_Headers.pretty
Parts:
- GND1, GND2, GND3, VCC1, VDD1: value INTERCONNECT_16X1 -> INTERCONNECT_1X16; symbol INTERCONNECT_16X1 -> INTERCONNECT_1X16
- J1, J10, J11, J12, J13, J14, J15, J16, J17, J18, J19, J2, J20, J21, J22, J23, J24, J25, J26, J27, J28, J29, J3, J30, J31, J32, J33, J34, J35, J36, J37, J38, J39, J4, J40, J41, J42, J43, J44, J45, J46, J47, J48, J49, J5, J50, J51, J52, J53, J54, J55, J56, J57, J58, J59, J6, J60, J61, J62, J63, J64, J7, J8, J9: value INTERCONNECT_3X1 -> INTERCONNECT_1X03; symbol INTERCONNECT_3X1 -> INTERCONNECT_1X03
- J65: value INTERCONNECT_2X1 -> INTERCONNECT_1X02; symbol INTERCONNECT_2X1 -> INTERCONNECT_1X02
Connections:
- net at C1.2, C2.2, GND1.1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: no longer U1.2 (GND)
